File: boards/MOM_KiCad/MOM.kicad_sch (KiCad schematic)
At the start: 27 parts, among them J1 JST-PH, J2 USB_C_Receptacle_USB2.0, Q1 DMG3415U, SW1 SW_Push, SW2 SW_Push, U1 AP2112K-3.3, U2 MCP73831-2-OT, U3 LC709204F, U4 ESP32-S3-MINI-1

Commit message: New schematic revision and repo cleanup
Parts:
- added C8: 2.2uF, symbol Device:C
- U1: value AP2112K-3.3 -> AP2112M-3.3; footprint Package_TO_SOT_SMD:SOT-23-5 -> Package_SO:Diodes_SO-8EP
Connections:
- net +3.3V: now also U1.1 (VOUT); no longer U1.5 (VOUT)
- net +BATT: now also U3.A4 (VDD); no longer U3.3 (VDD)
- net GND: now also U1.6 (GND), U1.7 (GND), U3.A2 (VSS), U3.B2 (TEST2), U3.C2 (TEST1), C8.2; no longer U1.2 (GND), U3.1 (TEST), U3.2 (VSS)
- net SCL: now also U3.B1 (SCL); no longer U3.8 (SCL)
- net SDA: now also U3.A1 (SDA); no longer U3.7 (SDA)
- net at D1.1 (K), Q1.2 (S), R2.1: now also U1.8 (VIN); no longer U1.1 (VIN)
- net at U1.3 (NC): no longer R2.2
- new net: R2.2, U1.5 (EN)
- new net: C8.1, U3.A3 (REG)
Other:
- moved on the sheet: D2, R2, R5, R6, U2

Commit message: Schematic updates
Parts:
- removed U3: LC709204F, Package_DFN_QFN:WDFN-8-1EP_4x3mm_P0.65mm_EP2.4x1.8mm, symbol Battery_Management:LC709203FQH-01TWG
- added C1: 10uF, Capacitor_Tantalum_SMD:CP_EIA-2012-12_Kemet-R_Pad1.30x1.05mm_HandSolder, symbol Device:C
- added C5: 0.1uF, Capacitor_Tantalum_SMD:CP_EIA-2012-12_Kemet-R_Pad1.30x1.05mm_HandSolder, symbol Device:C
- added U3: MAX17048G+T10, MAX17048G+T10:SON50P200X200X80-9N, symbol MAX17048G_T10:MAX17048G+T10
- C2: renamed from C1; footprint (none) -> Capacitor_Tantalum_SMD:CP_EIA-2012-12_Kemet-R_Pad1.30x1.05mm_HandSolder
- C3: renamed from C2; footprint (none) -> Capacitor_Tantalum_SMD:CP_EIA-2012-12_Kemet-R_Pad1.30x1.05mm_HandSolder
- C4: renamed from C3; footprint (none) -> Capacitor_Tantalum_SMD:CP_EIA-2012-12_Kemet-R_Pad1.30x1.05mm_HandSolder
- C6: renamed from C4; value 10uf -> 10uF; footprint (none) -> Capacitor_Tantalum_SMD:CP_EIA-2012-12_Kemet-R_Pad1.30x1.05mm_HandSolder
- C7: renamed from C5; value 10uf -> 10uF; footprint (none) -> Capacitor_Tantalum_SMD:CP_EIA-2012-12_Kemet-R_Pad1.30x1.05mm_HandSolder
- C8: renamed from C6; value 1uf -> 1uF; footprint (none) -> Capacitor_Tantalum_SMD:CP_EIA-2012-12_Kemet-R_Pad1.30x1.05mm_HandSolder
- C9: renamed from C7; footprint (none) -> Capacitor_Tantalum_SMD:CP_EIA-2012-12_Kemet-R_Pad1.30x1.05mm_HandSolder
- D1: value MBR0540 -> 5A/40V/550mV; footprint Diode_SMD:D_SOD-123 -> Package_SO:ONSemi_SO-8FL_488AA
- D2: value CHG -> AMBER; footprint (none) -> LED_THT:LED_D5.0mm
- D3: value PWR -> RED; footprint (none) -> LED_THT:LED_D5.0mm
- J1: footprint (none) -> Connector_JST:JST_PH_S2B-PH-K_1x02_P2.00mm_Horizontal
- J2: footprint (none) -> Connector_USB:USB_C_Receptacle_GCT_USB4085
- Q1: value DMG3415U -> DMP2045U
- R1, R2, R3, R4, R5, R7, R8: footprint (none) -> Resistor_SMD:R_1206_3216Metric_Pad1.30x1.75mm_HandSolder
- R6: value 5.1K -> 2K; footprint (none) -> Resistor_SMD:R_1206_3216Metric_Pad1.30x1.75mm_HandSolder
- SW1, SW2: footprint (none) -> Push_Button:SW_TS04-66-65-BK-160-SMT
Connections:
- net +BATT: now also C5.1, U3.2 (CELL), U3.3 (VDD)
- net GND: now also C1.2, C5.2, U3.1 (CTG), U3.4 (GND), U3.6 (QSTRT), U3.9 (EP); no longer C8.2
- net SCL: now also U3.7 (SCL)
- net SDA: now also U3.8 (SDA)
- net USB_D+: now also J2.B6 (D+)
- net USB_D-: now also J2.B7 (D-)
- net at D1.1 (K), Q1.2 (S), R2.1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: now also C1.1
- net U0TXD: no longer names the net of U4.39 (U0TXD/GPIO43/CLK_OUT1)
Other:
- moved on the sheet: D2, J1, R2, R5, R6, U2

Commit message: Franklin notebook updates
Parts:
- removed C8: 2.2uF, symbol Device:C
- C2, C3, C4, C6, C7, C8, C9: footprint Capacitor_Tantalum_SMD:CP_EIA-2012-12_Kemet-R_Pad1.30x1.05mm_HandSolder -> Capacitor_Tantalum_SMD:CP_EIA-2012-12_Kemet-R_Pad1.30x1.05mm_HandSolderCapacitor_Tantalum_SMD:CP_EIA-2012-12_Kemet-R_Pa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
- D1: footprint Package_SO:ONSemi_SO-8FL_488AA -> Library:D_SMBF_Handsoldering
- D3: footprint LED_THT:LED_D5.0mm -> LED_THT:LED_D5.0mmLED_THT:LED_D5.0mm
- J2: footprint Connector_USB:USB_C_Receptacle_GCT_USB4085 -> Connector_USB:USB_C_Receptacle_GCT_USB4085Connector_USB:USB_C_Receptacle_GCT_USB4085
- Q1: footprint Package_TO_SOT_SMD:SOT-23 -> Package_TO_SOT_SMD:SOT-23_Handsoldering
- R1, R3, R4, R7, R8: footprint Resistor_SMD:R_1206_3216Metric_Pad1.30x1.75mm_HandSolder -> Resistor_SMD:R_1206_3216Metric_Pad1.30x1.75mm_HandSolderResistor_SMD:R_1206_3216Metric_Pad1.30x1.75mm_HandSolder
- SW1, SW2: footprint Push_Button:SW_TS04-66-65-BK-160-SMT -> Push_Button:SW_TS04-66-65-BK-160-SMTPush_Button:SW_TS04-66-65-BK-160-SMT
- U2: value MCP73831-2-OT -> MCP73831; footprint Package_TO_SOT_SMD:SOT-23-5 -> MCP73831-MC:SON50P200X300X100-9N
- U4: footprint Espressif:ESP32-S3-MINI-1 -> ESP32:ESP32-S3-MINI-1

Commit message: PCB version alpha
Parts:
- added C10: 10uF, Capacitor_Tantalum_SMD:CP_EIA-2012-12_Kemet-R_Pad1.30x1.05mm_HandSolder, symbol Device:C
- added H1, H2, H3, H4: MountingHole, MountingHole:MountingHole_3.2mm_M3, symbol Mechanical:MountingHole
- C2, C3, C4, C6, C7, C8, C9: footprint Capacitor_Tantalum_SMD:CP_EIA-2012-12_Kemet-R_Pad1.30x1.05mm_HandSolderCapacitor_Tantalum_SMD:CP_EIA-2012-12_Kemet-R_Pa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 -> Capacitor_Tantalum_SMD:CP_EIA-2012-12_Kemet-R_Pad1.30x1.05mm_HandSolder
- D1: footprint Library:D_SMBF_Handsoldering -> SMBF:D_SMBF_Handsoldering
- D3: footprint LED_THT:LED_D5.0mmLED_THT:LED_D5.0mm -> LED_THT:LED_D5.0mm
- J2: footprint Connector_USB:USB_C_Receptacle_GCT_USB4085Connector_USB:USB_C_Receptacle_GCT_USB4085 -> Connector_USB:USB_C_Receptacle_GCT_USB4085
- R1, R3, R4, R7, R8: footprint Resistor_SMD:R_1206_3216Metric_Pad1.30x1.75mm_HandSolderResistor_SMD:R_1206_3216Metric_Pad1.30x1.75mm_HandSolder -> Resistor_SMD:R_1206_3216Metric_Pad1.30x1.75mm_HandSolder
- SW1, SW2: footprint Push_Button:SW_TS04-66-65-BK-160-SMTPush_Button:SW_TS04-66-65-BK-160-SMT -> Push_Button:SW_TS04-66-65-BK-160-SMT
- U1: footprint Package_SO:Diodes_SO-8EP -> AP2112M:Diodes_SO-8
Connections:
- net +BATT: now also U2.4 (VBAT), C10.1
- net GND: now also J2.S1 (SHIELD), U2.6 (VSS), U2.9 (EP), C10.2; no longer U2.2 (VSS)
- net VBUS: now also U2.1 (VDD), U2.2 (VDD); no longer U2.4 (VDD)
- net at R6.1: now also U2.8 (PROG); no longer U2.5 (PROG)
- net at D2.1 (K): now also R5.2; no longer R5.1
- new net: R5.1, U2.5 (STAT)
Other:
- moved on the sheet: D2, R5, R6
